File: RAILbooster.brd (EAGLE design)
At the start: 83.8 x 71.1 mm, 55 parts, among them IC1 LMD18200, IC3 LT1084, IC4 74HC10, IC5 SFH6731SMD8-OPT7, IC6 74HC4538, IC8 LM358D, IC9 LD117ADT50TR, J1 POWER_JACKPTH, X1 SCREWTERMINAL-5.08-2, X3 SCREWTERMINAL-5.08-2, X4 SCREWTERMINAL-5.08-2

Commit message: RAILbooster-2012-10-05
Parts:
- removed JP7, JP8: FIDUCIAL1.5X3, SparkFun:FIDUCIAL-1.5X3
- added C15, C22: 47uF, rcl:C0402
- added C16, C23: 10uF, rcl:C0402
- added C17, C19, C20, C21, C24, C26, C27, C28: .1uF, rcl:C0402
- added C18, C25: .01uF, rcl:C0402
- added D1, D2, D3, D4, D5, D6, D7, D8: (no value), Railstars:SOD-323
- added IC$1, IC$2: TPS715XX, Railstars:SC70
- added IC2, IC7: LV8402GP, Railstars:VCT24(3.5X3.5)
- added J2, J3: AVR_SPI_PRG_6NS, SparkFun-Connectors:2X3-NS
- added JP10, JP11, JP12, JP9: (no value), SparkFun-Connectors:1X02
- added R12, R13, R16, R17, R18, R19, R22, R23: 100K, rcl:R0402
- added R14, R15, R20, R21: 3.3K, rcl:R0402
- added U$12, U$24: ATTINY84A-MMH, Railstars:VQFN-20
- added U$13, U$25: DMN65D8LDW, Railstars:SOT363
- added U$14, U$15, U$16, U$17, U$18, U$19, U$20, U$26, U$27, U$28, U$29, U$30, U$31, U$32: PAD1MM, Railstars:LED_SOLDER_PAD
- added U$5, U$6, U$7, U$8: FIDUCIAL, adafruit:FIDUCIAL_1MM
- JP1, JP6: value FIDUCIAL1.5X3 -> M01SMDNS; device SparkFun:FIDUCIAL-1.5X3 -> SparkFun-Connectors:1X01NS
- moved JP1 69.3 mm to (52.1, 67.3)
- moved JP6 23.9 mm to (52.1, 62.2)
- moved R11 20.1 mm to (26.7, 5.08), turned to 0 degrees
- moved C14 2.54 mm to (17.8, 24.1)
- moved R10 2.54 mm to (17.8, 27.9)
- moved LED1 2.54 mm to (6.35, 33.0)
- moved LED2 2.54 mm to (6.35, 25.4)
- moved LED3 2.54 mm to (6.35, 17.8)
- moved LED4 2.54 mm to (6.35, 10.2)
- moved RN1 2.54 mm to (11.4, 25.4)
Connections:
- new net L2_1_!RESET: J2.5, U$12.P$13
- new net L2_1_5V: C15.1, C17.1, C19.1, IC$1.5, IC2.P$13, J2.2, U$12.P$9
- new net L2_1_BEMF: C20.1, R12.2, R13.1, U$12.P$2
- new net L2_1_DCC_L: D1.1, D2.2, R14.2, U$18.P$1
- new net L2_1_DCC_L_LL: R14.1, U$12.P$3
- new net L2_1_DCC_R: D3.2, D4.1, R15.2, U$19.P$1
- new net L2_1_DCC_R_LL: R15.1, U$12.P$4
- new net L2_1_ENABLE: IC2.P$12, IC2.P$16, U$12.P$12
- new net L2_1_F0: U$13.P$4, U$15.P$1
- new net L2_1_F1: U$13.P$1, U$14.P$1
- new net L2_1_FORWARD: IC2.P$10, IC2.P$14, U$12.P$15
- new net L2_1_GND: C15.2, C16.2, C17.2, C19.2, C20.2, C21.1, D1.2, D4.2, IC$1.2, IC2.P$17, IC2.P$18, IC2.P$3, IC2.P$4, J2.6, R16.2, R17.2, U$12.P$21, U$12.P$8, U$13.P$3, U$13.P$6
- new net L2_1_MISO: J2.1, R17.1, U$12.P$20, U$13.P$2
- new net L2_1_MOSI: J2.4, R16.1, U$12.P$16, U$13.P$5
- new net L2_1_MOTOR_L: IC2.P$2, IC2.P$6, R13.2, U$17.P$1
- new net L2_1_MOTOR_R: IC2.P$1, IC2.P$5, R12.1, U$16.P$1
- new net L2_1_N$1: C21.2, IC2.P$21
- new net L2_1_N$3: C18.1, IC2.P$19
- new net L2_1_N$9: C18.2, IC2.P$20
- new net L2_1_REVERSE: IC2.P$11, IC2.P$15, U$12.P$14
- new net L2_1_SCK: J2.3, U$12.P$1
- new net L2_1_VDCC: C16.1, D2.1, D3.1, IC$1.4, IC2.P$22, IC2.P$23, IC2.P$8, IC2.P$9, U$20.P$1
- new net L2_2_!RESET: J3.5, U$24.P$13
- new net L2_2_5V: C22.1, C24.1, C26.1, IC$2.5, IC7.P$13, J3.2, U$24.P$9
- new net L2_2_BEMF: C27.1, R18.2, R19.1, U$24.P$2
- new net L2_2_DCC_L: D5.1, D6.2, R20.2, U$30.P$1
- new net L2_2_DCC_L_LL: R20.1, U$24.P$3
- new net L2_2_DCC_R: D7.2, D8.1, R21.2, U$31.P$1
- new net L2_2_DCC_R_LL: R21.1, U$24.P$4
- new net L2_2_ENABLE: IC7.P$12, IC7.P$16, U$24.P$12
- new net L2_2_F0: U$25.P$4, U$27.P$1
- new net L2_2_F1: U$25.P$1, U$26.P$1
- new net L2_2_FORWARD: IC7.P$10, IC7.P$14, U$24.P$15
- new net L2_2_GND: C22.2, C23.2, C24.2, C26.2, C27.2, C28.1, D5.2, D8.2, IC$2.2, IC7.P$17, IC7.P$18, IC7.P$3, IC7.P$4, J3.6, R22.2, R23.2, U$24.P$21, U$24.P$8, U$25.P$3, U$25.P$6
- new net L2_2_MISO: J3.1, R23.1, U$24.P$20, U$25.P$2
- new net L2_2_MOSI: J3.4, R22.1, U$24.P$16, U$25.P$5
- new net L2_2_MOTOR_L: IC7.P$2, IC7.P$6, R19.2, U$29.P$1
- new net L2_2_MOTOR_R: IC7.P$1, IC7.P$5, R18.1, U$28.P$1
- new net L2_2_N$1: C28.2, IC7.P$21
- new net L2_2_N$3: C25.1, IC7.P$19
- new net L2_2_N$9: C25.2, IC7.P$20
- new net L2_2_REVERSE: IC7.P$11, IC7.P$15, U$24.P$14
- new net L2_2_SCK: J3.3, U$24.P$1
- new net L2_2_VDCC: C23.1, D6.1, D7.1, IC$2.4, IC7.P$22, IC7.P$23, IC7.P$8, IC7.P$9, U$32.P$1
- net !DCC_MISSING: now also JP11.1
- net FAULT: now also JP12.1
- net GND: now also JP1.1, JP10.2, JP11.2, JP12.2, JP9.2
- net N$1: now also JP6.1
- net VCC: now also JP10.1
- net VDD: now also JP9.1
Routing:
- net L2_2_5V: track 0.00 -> 29.5 mm, vias 0 -> 3
- net L2_1_5V: track 0.00 -> 29.5 mm, vias 0 -> 3
- net L2_2_VDCC: track 0.00 -> 24.6 mm, vias 0 -> 5
- net L2_1_VDCC: track 0.00 -> 24.6 mm, vias 0 -> 5
- net N$13: track 4.06 -> 27.6 mm, vias 0 -> 2
- net L2_2_MOSI: track 0.00 -> 21.1 mm, vias 0 -> 1
- net L2_1_MOSI: track 0.00 -> 21.1 mm, vias 0 -> 1
- net L2_1_MISO: track 0.00 -> 20.6 mm, vias 0 -> 2
- net L2_2_MISO: track 0.00 -> 20.6 mm, vias 0 -> 2
- net L2_1_BEMF: track 0.00 -> 16.5 mm, vias 0 -> 3
- net L2_2_BEMF: track 0.00 -> 16.5 mm, vias 0 -> 3
- net L2_2_DCC_R: track 0.00 -> 16.0 mm, vias 0 -> 4
- net L2_1_DCC_R: track 0.00 -> 16.0 mm, vias 0 -> 4
- net L2_1_!RESET: track 0.00 -> 13.6 mm, vias 0 -> 1
- net L2_2_!RESET: track 0.00 -> 13.6 mm, vias 0 -> 1
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- added copper zone on layer 1, net L2_1_GND
- added copper zone on layer 16, net L2_1_GND
- added copper zone on layer 1, net L2_2_GND
- added copper zone on layer 16, net L2_2_GND
Other:
- board size 83.8 x 71.1 mm -> 83.8 x 86.4 mm
- board text added: "+"
- board text added: "100003268"
- board text added: "L2-P"
- board text added: "REV B 2012-10-05"
- board text added: "railstars"
- board text removed: "44761"
- board text removed: "REV A 2012-01-15"

Commit message: Railbooster 20121005 Final
Parts:
- removed C15, C22: 47uF, rcl:C0402
- removed C16, C23: 10uF, rcl:C0402
- removed C17, C19, C20, C21, C24, C26, C27, C28: .1uF, rcl:C0402
- removed C18, C25: .01uF, rcl:C0402
- removed D1, D2, D3, D4, D5, D6, D7, D8: (no value), Railstars:SOD-323
- removed IC$1, IC$2: TPS715XX, Railstars:SC70
- removed IC2, IC7: LV8402GP, Railstars:VCT24(3.5X3.5)
- removed J2, J3: AVR_SPI_PRG_6NS, SparkFun-Connectors:2X3-NS
- removed R12, R13, R16, R17, R18, R19, R22, R23: 100K, rcl:R0402
- removed R14, R15, R20, R21: 3.3K, rcl:R0402
- removed U$12, U$24: ATTINY84A-MMH, Railstars:VQFN-20
- removed U$13, U$25: DMN65D8LDW, Railstars:SOT363
- removed U$14, U$15, U$16, U$17, U$18, U$19, U$20, U$26, U$27, U$28, U$29, U$30, U$31, U$32: PAD1MM, Railstars:LED_SOLDER_PAD
Connections:
- removed net L2_1_!RESET: J2.5, U$12.P$13
- removed net L2_1_5V: C15.1, C17.1, C19.1, IC$1.5, IC2.P$13, J2.2, U$12.P$9
- removed net L2_1_BEMF: C20.1, R12.2, R13.1, U$12.P$2
- removed net L2_1_DCC_L: D1.1, D2.2, R14.2, U$18.P$1
- removed net L2_1_DCC_L_LL: R14.1, U$12.P$3
- removed net L2_1_DCC_R: D3.2, D4.1, R15.2, U$19.P$1
- removed net L2_1_DCC_R_LL: R15.1, U$12.P$4
- removed net L2_1_ENABLE: IC2.P$12, IC2.P$16, U$12.P$12
- removed net L2_1_F0: U$13.P$4, U$15.P$1
- removed net L2_1_F1: U$13.P$1, U$14.P$1
- removed net L2_1_FORWARD: IC2.P$10, IC2.P$14, U$12.P$15
- removed net L2_1_GND: C15.2, C16.2, C17.2, C19.2, C20.2, C21.1, D1.2, D4.2, IC$1.2, IC2.P$17, IC2.P$18, IC2.P$3, IC2.P$4, J2.6, R16.2, R17.2, U$12.P$21, U$12.P$8, U$13.P$3, U$13.P$6
- removed net L2_1_MISO: J2.1, R17.1, U$12.P$20, U$13.P$2
- removed net L2_1_MOSI: J2.4, R16.1, U$12.P$16, U$13.P$5
- removed net L2_1_MOTOR_L: IC2.P$2, IC2.P$6, R13.2, U$17.P$1
- removed net L2_1_MOTOR_R: IC2.P$1, IC2.P$5, R12.1, U$16.P$1
- removed net L2_1_N$1: C21.2, IC2.P$21
- removed net L2_1_N$3: C18.1, IC2.P$19
- removed net L2_1_N$9: C18.2, IC2.P$20
- removed net L2_1_REVERSE: IC2.P$11, IC2.P$15, U$12.P$14
- removed net L2_1_SCK: J2.3, U$12.P$1
- removed net L2_1_VDCC: C16.1, D2.1, D3.1, IC$1.4, IC2.P$22, IC2.P$23, IC2.P$8, IC2.P$9, U$20.P$1
- removed net L2_2_!RESET: J3.5, U$24.P$13
- removed net L2_2_5V: C22.1, C24.1, C26.1, IC$2.5, IC7.P$13, J3.2, U$24.P$9
- removed net L2_2_BEMF: C27.1, R18.2, R19.1, U$24.P$2
- removed net L2_2_DCC_L: D5.1, D6.2, R20.2, U$30.P$1
- removed net L2_2_DCC_L_LL: R20.1, U$24.P$3
- removed net L2_2_DCC_R: D7.2, D8.1, R21.2, U$31.P$1
- removed net L2_2_DCC_R_LL: R21.1, U$24.P$4
- removed net L2_2_ENABLE: IC7.P$12, IC7.P$16, U$24.P$12
- removed net L2_2_F0: U$25.P$4, U$27.P$1
- removed net L2_2_F1: U$25.P$1, U$26.P$1
- removed net L2_2_FORWARD: IC7.P$10, IC7.P$14, U$24.P$15
- removed net L2_2_GND: C22.2, C23.2, C24.2, C26.2, C27.2, C28.1, D5.2, D8.2, IC$2.2, IC7.P$17, IC7.P$18, IC7.P$3, IC7.P$4, J3.6, R22.2, R23.2, U$24.P$21, U$24.P$8, U$25.P$3, U$25.P$6
- removed net L2_2_MISO: J3.1, R23.1, U$24.P$20, U$25.P$2
- removed net L2_2_MOSI: J3.4, R22.1, U$24.P$16, U$25.P$5
- removed net L2_2_MOTOR_L: IC7.P$2, IC7.P$6, R19.2, U$29.P$1
- removed net L2_2_MOTOR_R: IC7.P$1, IC7.P$5, R18.1, U$28.P$1
- removed net L2_2_N$1: C28.2, IC7.P$21
- removed net L2_2_N$3: C25.1, IC7.P$19
- removed net L2_2_N$9: C25.2, IC7.P$20
- removed net L2_2_REVERSE: IC7.P$11, IC7.P$15, U$24.P$14
- removed net L2_2_SCK: J3.3, U$24.P$1
- removed net L2_2_VDCC: C23.1, D6.1, D7.1, IC$2.4, IC7.P$22, IC7.P$23, IC7.P$8, IC7.P$9, U$32.P$1
Routing:
- net L2_2_5V: track 29.5 -> 0.00 mm, vias 3 -> 0
- net L2_1_5V: track 29.5 -> 0.00 mm, vias 3 -> 0
- net L2_2_VDCC: track 24.6 -> 0.00 mm, vias 5 -> 0
- net L2_1_VDCC: track 24.6 -> 0.00 mm, vias 5 -> 0
- net L2_2_MOSI: track 21.1 -> 0.00 mm, vias 1 -> 0
- net L2_1_MOSI: track 21.1 -> 0.00 mm, vias 1 -> 0
- net L2_1_MISO: track 20.6 -> 0.00 mm, vias 2 -> 0
- net L2_2_MISO: track 20.6 -> 0.00 mm, vias 2 -> 0
- net L2_1_BEMF: track 16.5 -> 0.00 mm, vias 3 -> 0
- net L2_2_BEMF: track 16.5 -> 0.00 mm, vias 3 -> 0
- net L2_2_DCC_R: track 16.0 -> 0.00 mm, vias 4 -> 0
- net L2_1_DCC_R: track 16.0 -> 0.00 mm, vias 4 -> 0
- net L2_1_!RESET: track 13.6 -> 0.00 mm, vias 1 -> 0
- net L2_2_!RESET: track 13.6 -> 0.00 mm, vias 1 -> 0
- net L2_1_MOTOR_L: track 12.6 -> 0.00 mm, vias 3 -> 0
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- removed copper zone on layer 1, net L2_1_GND
- removed copper zone on layer 16, net L2_1_GND
- removed copper zone on layer 1, net L2_2_GND
- removed copper zone on layer 16, net L2_2_GND
Other:
- board size 83.8 x 86.4 mm -> 83.8 x 71.1 mm
- board text added: "Assembled in USA"
- board text removed: "100003268"
- board text removed: "Assembled in Colorado, USA"
- board text removed: "L2-P"
- board text removed: "railstars"
