File: RAILbooster.sch (EAGLE design)
At the start: 52 parts, among them IC1 LMD18200, IC3 LT1084, IC4 74HC10, IC5 SFH6731SMD8-OPT7, IC6 74HC4538, IC8 LM358D, IC9 LD117ADT50TR, J1 POWER_JACKPTH, X1 SCREWTERMINAL-5.08-2, X3 SCREWTERMINAL-5.08-2, X4 SCREWTERMINAL-5.08-2

Commit message: RAILbooster-2012-10-05
Parts:
- removed JP7, JP8: FIDUCIAL1.5X3, SparkFun:FIDUCIAL1.5X3
- added C15, C22: 47uF, rcl:C-USC0402
- added C16, C23: 10uF, rcl:C-USC0402
- added C17, C19, C20, C21, C24, C26, C27, C28: .1uF, rcl:C-USC0402
- added C18, C25: .01uF, rcl:C-USC0402
- added D1, D2, D3, D4, D5, D6, D7, D8: (no value), Railstars:DIODESOD
- added IC$1, IC$2: TPS715XX, Railstars:TPS715XX
- added IC2, IC7: LV8402GP, Railstars:LV8402GP
- added J2, J3: AVR_SPI_PRG_6NS, SparkFun-Connectors:AVR_SPI_PRG_6NS
- added JP10, JP11, JP12, JP9: (no value), SparkFun-Connectors:M02PTH
- added R12, R13, R16, R17, R18, R19, R22, R23: 100K, rcl:R-US_R0402
- added R14, R15, R20, R21: 3.3K, rcl:R-US_R0402
- added U$12, U$24: ATTINY84A-MMH, Railstars:ATTINY84A-MMH
- added U$13, U$25: DMN65D8LDW, Railstars:DMN65D8LDW
- added U$14, U$15, U$16, U$17, U$18, U$19, U$20, U$26, U$27, U$28, U$29, U$30, U$31, U$32: PAD1MM, Railstars:PAD1MM
- added U$5, U$6, U$7, U$8: FIDUCIAL, adafruit:FIDUCIAL
- JP1, JP6: value FIDUCIAL1.5X3 -> M01SMDNS; device SparkFun:FIDUCIAL1.5X3 -> SparkFun-Connectors:M01SMDNS
Connections:
- new net L2_1_!RESET: J2.5, U$12.!RESET
- new net L2_1_5V: C15.1, C17.1, C19.1, IC$1.OUT, IC2.VCC, J2.2, U$12.VCC
- new net L2_1_BEMF: C20.1, R12.2, R13.1, U$12.PA3/ADC3
- new net L2_1_DCC_L: D1.C, D2.A, R14.2, U$18.P$1
- new net L2_1_DCC_L_LL: R14.1, U$12.PA2/ADC2
- new net L2_1_DCC_R: D3.A, D4.C, R15.2, U$19.P$1
- new net L2_1_DCC_R_LL: R15.1, U$12.PA1/ADC1
- new net L2_1_ENABLE: IC2.EN1, IC2.EN2, U$12.PB1
- new net L2_1_F0: U$13G$1.D, U$15.P$1
- new net L2_1_F1: U$13G$2.D, U$14.P$1
- new net L2_1_FORWARD: IC2.IN2, IC2.IN4, U$12.PA7/OC0B
- new net L2_1_GND: C15.2, C16.2, C17.2, C19.2, C20.2, C21.1, D1.A, D4.A, IC$1.GND, IC2.EXTRA, IC2.PGND, IC2.SGND, J2.6, R16.2, R17.2, U$12.GND, U$13G$1.S, U$13G$2.S
- new net L2_1_MISO: J2.1, R17.1, U$12.PA5/OC1B, U$13G$1.G
- new net L2_1_MOSI: J2.4, R16.1, U$12.PA6/OC1A, U$13G$2.G
- new net L2_1_MOTOR_L: IC2.OUT2, IC2.OUT4, R13.2, U$17.P$1
- new net L2_1_MOTOR_R: IC2.OUT1, IC2.OUT3, R12.1, U$16.P$1
- new net L2_1_N$1: C21.2, IC2.VG
- new net L2_1_N$3: C18.1, IC2.C1L
- new net L2_1_N$9: C18.2, IC2.C1H
- new net L2_1_REVERSE: IC2.IN1, IC2.IN3, U$12.PB2/OC0A
- new net L2_1_SCK: J2.3, U$12.PA4/ADC4
- new net L2_1_VDCC: C16.1, D2.C, D3.C, IC$1.IN, IC2.VM, U$20.P$1
- new net L2_2_!RESET: J3.5, U$24.!RESET
- new net L2_2_5V: C22.1, C24.1, C26.1, IC$2.OUT, IC7.VCC, J3.2, U$24.VCC
- new net L2_2_BEMF: C27.1, R18.2, R19.1, U$24.PA3/ADC3
- new net L2_2_DCC_L: D5.C, D6.A, R20.2, U$30.P$1
- new net L2_2_DCC_L_LL: R20.1, U$24.PA2/ADC2
- new net L2_2_DCC_R: D7.A, D8.C, R21.2, U$31.P$1
- new net L2_2_DCC_R_LL: R21.1, U$24.PA1/ADC1
- new net L2_2_ENABLE: IC7.EN1, IC7.EN2, U$24.PB1
- new net L2_2_F0: U$25G$1.D, U$27.P$1
- new net L2_2_F1: U$25G$2.D, U$26.P$1
- new net L2_2_FORWARD: IC7.IN2, IC7.IN4, U$24.PA7/OC0B
- new net L2_2_GND: C22.2, C23.2, C24.2, C26.2, C27.2, C28.1, D5.A, D8.A, IC$2.GND, IC7.EXTRA, IC7.PGND, IC7.SGND, J3.6, R22.2, R23.2, U$24.GND, U$25G$1.S, U$25G$2.S
- new net L2_2_MISO: J3.1, R23.1, U$24.PA5/OC1B, U$25G$1.G
- new net L2_2_MOSI: J3.4, R22.1, U$24.PA6/OC1A, U$25G$2.G
- new net L2_2_MOTOR_L: IC7.OUT2, IC7.OUT4, R19.2, U$29.P$1
- new net L2_2_MOTOR_R: IC7.OUT1, IC7.OUT3, R18.1, U$28.P$1
- new net L2_2_N$1: C28.2, IC7.VG
- new net L2_2_N$3: C25.1, IC7.C1L
- new net L2_2_N$9: C25.2, IC7.C1H
- new net L2_2_REVERSE: IC7.IN1, IC7.IN3, U$24.PB2/OC0A
- new net L2_2_SCK: J3.3, U$24.PA4/ADC4
- new net L2_2_VDCC: C23.1, D6.C, D7.C, IC$2.IN, IC7.VM, U$32.P$1
- net !DCC_MISSING: now also JP11.1
- net FAULT: now also JP12.1
- net GND: now also JP1.1, JP10.2, JP11.2, JP12.2, JP9.2
- net N$1: now also JP6.1
- net VCC: now also JP10.1
- net VDD: now also JP9.1

Commit message: Railbooster 20121005 Final
Parts:
- removed C15, C22: 47uF, rcl:C-USC0402
- removed C16, C23: 10uF, rcl:C-USC0402
- removed C17, C19, C20, C21, C24, C26, C27, C28: .1uF, rcl:C-USC0402
- removed C18, C25: .01uF, rcl:C-USC0402
- removed D1, D2, D3, D4, D5, D6, D7, D8: (no value), Railstars:DIODESOD
- removed IC$1, IC$2: TPS715XX, Railstars:TPS715XX
- removed IC2, IC7: LV8402GP, Railstars:LV8402GP
- removed J2, J3: AVR_SPI_PRG_6NS, SparkFun-Connectors:AVR_SPI_PRG_6NS
- removed R12, R13, R16, R17, R18, R19, R22, R23: 100K, rcl:R-US_R0402
- removed R14, R15, R20, R21: 3.3K, rcl:R-US_R0402
- removed U$12, U$24: ATTINY84A-MMH, Railstars:ATTINY84A-MMH
- removed U$13, U$25: DMN65D8LDW, Railstars:DMN65D8LDW
- removed U$14, U$15, U$16, U$17, U$18, U$19, U$20, U$26, U$27, U$28, U$29, U$30, U$31, U$32: PAD1MM, Railstars:PAD1MM
Connections:
- removed net L2_1_!RESET: J2.5, U$12.!RESET
- removed net L2_1_5V: C15.1, C17.1, C19.1, IC$1.OUT, IC2.VCC, J2.2, U$12.VCC
- removed net L2_1_BEMF: C20.1, R12.2, R13.1, U$12.PA3/ADC3
- removed net L2_1_DCC_L: D1.C, D2.A, R14.2, U$18.P$1
- removed net L2_1_DCC_L_LL: R14.1, U$12.PA2/ADC2
- removed net L2_1_DCC_R: D3.A, D4.C, R15.2, U$19.P$1
- removed net L2_1_DCC_R_LL: R15.1, U$12.PA1/ADC1
- removed net L2_1_ENABLE: IC2.EN1, IC2.EN2, U$12.PB1
- removed net L2_1_F0: U$13G$1.D, U$15.P$1
- removed net L2_1_F1: U$13G$2.D, U$14.P$1
- removed net L2_1_FORWARD: IC2.IN2, IC2.IN4, U$12.PA7/OC0B
- removed net L2_1_GND: C15.2, C16.2, C17.2, C19.2, C20.2, C21.1, D1.A, D4.A, IC$1.GND, IC2.EXTRA, IC2.PGND, IC2.SGND, J2.6, R16.2, R17.2, U$12.GND, U$13G$1.S, U$13G$2.S
- removed net L2_1_MISO: J2.1, R17.1, U$12.PA5/OC1B, U$13G$1.G
- removed net L2_1_MOSI: J2.4, R16.1, U$12.PA6/OC1A, U$13G$2.G
- removed net L2_1_MOTOR_L: IC2.OUT2, IC2.OUT4, R13.2, U$17.P$1
- removed net L2_1_MOTOR_R: IC2.OUT1, IC2.OUT3, R12.1, U$16.P$1
- removed net L2_1_N$1: C21.2, IC2.VG
- removed net L2_1_N$3: C18.1, IC2.C1L
- removed net L2_1_N$9: C18.2, IC2.C1H
- removed net L2_1_REVERSE: IC2.IN1, IC2.IN3, U$12.PB2/OC0A
- removed net L2_1_SCK: J2.3, U$12.PA4/ADC4
- removed net L2_1_VDCC: C16.1, D2.C, D3.C, IC$1.IN, IC2.VM, U$20.P$1
- removed net L2_2_!RESET: J3.5, U$24.!RESET
- removed net L2_2_5V: C22.1, C24.1, C26.1, IC$2.OUT, IC7.VCC, J3.2, U$24.VCC
- removed net L2_2_BEMF: C27.1, R18.2, R19.1, U$24.PA3/ADC3
- removed net L2_2_DCC_L: D5.C, D6.A, R20.2, U$30.P$1
- removed net L2_2_DCC_L_LL: R20.1, U$24.PA2/ADC2
- removed net L2_2_DCC_R: D7.A, D8.C, R21.2, U$31.P$1
- removed net L2_2_DCC_R_LL: R21.1, U$24.PA1/ADC1
- removed net L2_2_ENABLE: IC7.EN1, IC7.EN2, U$24.PB1
- removed net L2_2_F0: U$25G$1.D, U$27.P$1
- removed net L2_2_F1: U$25G$2.D, U$26.P$1
- removed net L2_2_FORWARD: IC7.IN2, IC7.IN4, U$24.PA7/OC0B
- removed net L2_2_GND: C22.2, C23.2, C24.2, C26.2, C27.2, C28.1, D5.A, D8.A, IC$2.GND, IC7.EXTRA, IC7.PGND, IC7.SGND, J3.6, R22.2, R23.2, U$24.GND, U$25G$1.S, U$25G$2.S
- removed net L2_2_MISO: J3.1, R23.1, U$24.PA5/OC1B, U$25G$1.G
- removed net L2_2_MOSI: J3.4, R22.1, U$24.PA6/OC1A, U$25G$2.G
- removed net L2_2_MOTOR_L: IC7.OUT2, IC7.OUT4, R19.2, U$29.P$1
- removed net L2_2_MOTOR_R: IC7.OUT1, IC7.OUT3, R18.1, U$28.P$1
- removed net L2_2_N$1: C28.2, IC7.VG
- removed net L2_2_N$3: C25.1, IC7.C1L
- removed net L2_2_N$9: C25.2, IC7.C1H
- removed net L2_2_REVERSE: IC7.IN1, IC7.IN3, U$24.PB2/OC0A
- removed net L2_2_SCK: J3.3, U$24.PA4/ADC4
- removed net L2_2_VDCC: C23.1, D6.C, D7.C, IC$2.IN, IC7.VM, U$32.P$1
